File: kicad/key_matrix.kicad_sch (KiCad schematic)
At the start: 127 parts, among them SW1 SW_Push, SW10 SW_Push, SW11 SW_Push, SW12 SW_Push, SW13 SW_Push, SW14 SW_Push, SW15 SW_Push, SW16 SW_Push, SW17 SW_Push, SW18 SW_Push, SW19 SW_Push, SW2 SW_Push, SW20 SW_Push, SW21 SW_Push, SW22 SW_Push, SW23 SW_Push, SW24 SW_Push, SW25 SW_Push, SW26 SW_Push, SW27 SW_Push, SW28 SW_Push, SW29 SW_Push, SW3 SW_Push, SW30 SW_Push, SW31 SW_Push, SW32 SW_Push, SW33 SW_Push, SW34 SW_Push, SW35 SW_Push, SW36 SW_Push, SW37 SW_Push, SW38 SW_Push, SW39 SW_Push, SW4 SW_Push, SW40 SW_Push, SW41 SW_Push, SW42 SW_Push, SW43 SW_Push, SW44 SW_Push, SW45 SW_Push, SW46 SW_Push, SW47 SW_Push, SW48 SW_Push, SW49 SW_Push, SW5 SW_Push, SW50 SW_Push, SW51 SW_Push, SW52 SW_Push, SW53 SW_Push, SW54 SW_Push, SW55 SW_Push, SW56 SW_Push, SW57 SW_Push, SW58 SW_Push, SW59 SW_Push, SW6 SW_Push, SW60 SW_Push, SW61 SW_Push, SW7 SW_Push, SW8 SW_Push, SW9 SW_Push

Commit message: schematics done
Parts:
- SW1, SW10, SW11, SW12, SW13, SW14, SW15, SW16, SW17, SW18, SW19, SW2, SW20, SW21, SW22, SW23, SW24, SW25, SW26, SW27, SW28, SW29, SW3, SW30, SW31, SW32, SW33, SW34, SW35, SW36, SW37, SW38, SW39, SW4, SW40, SW41, SW42, SW43, SW44, SW45, SW46, SW47, SW48, SW49, SW5, SW50, SW51, SW52, SW53, SW54, SW55, SW56, SW57, SW58, SW59, SW6, SW60, SW61, SW7, SW8, SW9: footprint PCM_marbastlib-mx:SW_MX_1u -> PCM_marbastlib-mx:SW_MX_HS_CPG151101S11_1u
- renumbered D62 to D1, D71 to D10, D72 to D11, D73 to D12, D74 to D13, D75 to D14, D76 to D15, D77 to D16, D78 to D17, D79 to D18, D80 to D19, D63 to D2, D81 to D20, D82 to D21, D83 to D22, D84 to D23, D85 to D24, D86 to D25, D87 to D26, D88 to D27, D89 to D28, D90 to D29, D64 to D3, D91 to D30, D92 to D31, D93 to D32, D94 to D33, D95 to D34, D96 to D35, D97 to D36, D98 to D37, D99 to D38, D100 to D39, D65 to D4, D101 to D40, D102 to D41, D103 to D42, D104 to D43, D105 to D44, D106 to D45, D107 to D46, D108 to D47, D109 to D48, D110 to D49, D66 to D5, D111 to D50, D112 to D51, D113 to D52, D114 to D53, D115 to D54, D116 to D55, D117 to D56, D118 to D57, D119 to D58, D120 to D59, D67 to D6, D121 to D60, D122 to D61, D68 to D7, D69 to D8, D70 to D9
