File: kicad/kicad.kicad_pcb (KiCad board)
At the start: 2 copper layers, 128 parts, among them SW1 SW_Push, SW10 SW_Push, SW11 SW_Push, SW12 SW_Push, SW13 SW_Push, SW14 SW_Push, SW15 SW_Push, SW16 SW_Push, SW17 SW_Push, SW18 SW_Push, SW19 SW_Push, SW2 SW_Push, SW20 SW_Push, SW21 SW_Push, SW22 SW_Push, SW23 SW_Push, SW24 SW_Push, SW25 SW_Push, SW26 SW_Push, SW27 SW_Push, SW28 SW_Push, SW29 SW_Push, SW3 SW_Push, SW30 SW_Push, SW31 SW_Push, SW32 SW_Push, SW33 SW_Push, SW34 SW_Push, SW35 SW_Push, SW36 SW_Push, SW37 SW_Push, SW38 SW_Push, SW39 SW_Push, SW4 SW_Push, SW40 SW_Push, SW41 SW_Push, SW42 SW_Push, SW43 SW_Push, SW44 SW_Push, SW45 SW_Push, SW46 SW_Push, SW47 SW_Push, SW48 SW_Push, SW49 SW_Push, SW5 SW_Push, SW50 SW_Push, SW51 SW_Push, SW52 SW_Push, SW53 SW_Push, SW54 SW_Push, SW55 SW_Push, SW56 SW_Push, SW57 SW_Push, SW58 SW_Push, SW59 SW_Push, SW6 SW_Push, SW60 SW_Push, SW61 SW_Push, SW7 SW_Push, SW8 SW_Push, SW9 SW_Push

Commit message: restarting again aaa
Parts:
- added D62: 1N4148, Diode_THT:D_DO-35_SOD27_P7.62mm_Horizontal, F.Cu at (249.5, 181.3)
- D1: value 1N4148 -> SK6812MINI-E; footprint Diode_THT:D_DO-35_SOD27_P7.62mm_Horizontal -> LED_SMD:LED_SK6812MINI-E_3.2x2.8mm_P1.5mm_ReverseMount
- moved SW15 257.0 mm to (122.1, 152.8)
- moved SW14 234.3 mm to (122.1, 137.7)
- moved SW27 214.4 mm to (137.1, 197.9)
- moved SW29 212.7 mm to (152.2, 92.6)
- moved SW13 211.8 mm to (122.1, 122.7)
- moved D1 202.3 mm to (289.0, 72.4), turned to 0 degrees
- moved SW42 199.4 mm to (167.2, 152.8)
- moved D14 193.1 mm to (206.4, 195.5), turned to 0 degrees
- moved SW12 190.5 mm to (122.1, 107.6)
- moved SW26 188.3 mm to (137.1, 182.9), turned to 0 degrees
- moved SW28 187.8 mm to (152.2, 77.5)
- moved SW9 186.4 mm to (107.0, 197.9), turned to 0 degrees
- moved SW54 182.2 mm to (182.3, 197.9)
- moved D15 176.5 mm to (217.2, 152.9), turned to 0 degrees
- moved D13 176.5 mm to (206.4, 192.0), turned to 0 degrees
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Connections:
- A1 pad 13: unconnected-(A1-GND-Pad13)_1 -> GND
- A1 pad 18: unconnected-(A1-GND-Pad13)_6 -> GND
- A1 pad 23: unconnected-(A1-GND-Pad13)_2 -> GND
- A1 pad 26: unconnected-(A1-GPIO20-Pad26) -> /RGB
- A1 pad 28: unconnected-(A1-GND-Pad13)_4 -> GND
- A1 pad 3: unconnected-(A1-GND-Pad13) -> GND
- A1 pad 38: unconnected-(A1-GND-Pad13)_5 -> GND
- A1 pad 8: unconnected-(A1-GND-Pad13)_3 -> GND
- D1 pad 1: /ROW0 -> unconnected-(D1-VSS-Pad1)
- D1 pad 2: Net-(D1-A) -> unconnected-(D1-DIN-Pad2)
- D10 pad 1: /ROW0 -> /KEY_MATRIX/ROW3
- D11 pad 1: /ROW0 -> /KEY_MATRIX/ROW0
- D12 pad 1: /ROW0 -> /KEY_MATRIX/ROW1
- D13 pad 1: /ROW0 -> /KEY_MATRIX/ROW2
- D14 pad 1: /ROW0 -> /KEY_MATRIX/ROW3
- D15 pad 1: /ROW0 -> /KEY_MATRIX/ROW0
- D16 pad 1: /ROW1 -> /KEY_MATRIX/ROW1
- D17 pad 1: /ROW1 -> /KEY_MATRIX/ROW2
- D18 pad 1: /ROW1 -> /KEY_MATRIX/ROW3
- D19 pad 1: /ROW1 -> /KEY_MATRIX/ROW4
- D2 pad 1: /ROW0 -> /KEY_MATRIX/ROW0
- D20 pad 1: /ROW1 -> /KEY_MATRIX/ROW0
- D21 pad 1: /ROW1 -> /KEY_MATRIX/ROW1
- D22 pad 1: /ROW1 -> /KEY_MATRIX/ROW2
- D23 pad 1: /ROW1 -> /KEY_MATRIX/ROW3
- D24 pad 1: /ROW1 -> /KEY_MATRIX/ROW4
- D25 pad 1: /ROW1 -> /KEY_MATRIX/ROW0
- D26 pad 1: /ROW1 -> /KEY_MATRIX/ROW1
- D27 pad 1: /ROW1 -> /KEY_MATRIX/ROW2
- D28 pad 1: /ROW1 -> /KEY_MATRIX/ROW3
- D29 pad 1: /ROW1 -> /KEY_MATRIX/ROW4
- D3 pad 1: /ROW0 -> /KEY_MATRIX/ROW1
- D30 pad 1: /ROW2 -> /KEY_MATRIX/ROW0
- D31 pad 1: /ROW2 -> /KEY_MATRIX/ROW0
- D32 pad 1: /ROW2 -> /KEY_MATRIX/ROW1
- D33 pad 1: /ROW2 -> /KEY_MATRIX/ROW2
- D34 pad 1: /ROW2 -> /KEY_MATRIX/ROW3
- D35 pad 1: /ROW2 -> /KEY_MATRIX/ROW4
- D36 pad 1: /ROW2 -> /KEY_MATRIX/ROW0
- D37 pad 1: /ROW2 -> /KEY_MATRIX/ROW1
- D38 pad 1: /ROW2 -> /KEY_MATRIX/ROW2
- D39 pad 1: /ROW2 -> /KEY_MATRIX/ROW3
- D4 pad 1: /ROW0 -> /KEY_MATRIX/ROW2
- D40 pad 1: /ROW2 -> /KEY_MATRIX/ROW0
- D41 pad 1: /ROW2 -> /KEY_MATRIX/ROW1
- D42 pad 1: /ROW2 -> /KEY_MATRIX/ROW2
- D43 pad 1: /ROW3 -> /KEY_MATRIX/ROW3
- D44 pad 1: /ROW3 -> /KEY_MATRIX/ROW4
- D45 pad 1: /ROW3 -> /KEY_MATRIX/ROW0
- D46 pad 1: /ROW3 -> /KEY_MATRIX/ROW1
- D47 pad 1: /ROW3 -> /KEY_MATRIX/ROW2
- D48 pad 1: /ROW3 -> /KEY_MATRIX/ROW3
- D49 pad 1: /ROW3 -> /KEY_MATRIX/ROW0
- D5 pad 1: /ROW0 -> /KEY_MATRIX/ROW3
- D50 pad 1: /ROW3 -> /KEY_MATRIX/ROW1
- D51 pad 1: /ROW3 -> /KEY_MATRIX/ROW0
- D52 pad 1: /ROW3 -> /KEY_MATRIX/ROW1
- D53 pad 1: /ROW3 -> /KEY_MATRIX/ROW2
- D54 pad 1: /ROW3 -> /KEY_MATRIX/ROW3
- D55 pad 1: /ROW4 -> /KEY_MATRIX/ROW0
- D56 pad 1: /ROW4 -> /KEY_MATRIX/ROW1
- D57 pad 1: /ROW4 -> /KEY_MATRIX/ROW2
- D58 pad 1: /ROW4 -> /KEY_MATRIX/ROW0
- D59 pad 1: /ROW4 -> /KEY_MATRIX/ROW1
- D6 pad 1: /ROW0 -> /KEY_MATRIX/ROW4
- D60 pad 1: /ROW4 -> /KEY_MATRIX/ROW2
- D61 pad 1: /ROW4 -> /KEY_MATRIX/ROW3
- D7 pad 1: /ROW0 -> /KEY_MATRIX/ROW0
- D8 pad 1: /ROW0 -> /KEY_MATRIX/ROW1
- D9 pad 1: /ROW0 -> /KEY_MATRIX/ROW2
- SW1 pad 1: /COL0 -> /KEY_MATRIX/COL0
- SW1 pad 2: Net-(D1-A) -> Net-(D2-A)
- SW10 pad 1: /COL9 -> /KEY_MATRIX/COL2
- SW10 pad 2: Net-(D10-A) -> Net-(D11-A)
- SW11 pad 1: /COL10 -> /KEY_MATRIX/COL2
- SW11 pad 2: Net-(D11-A) -> Net-(D12-A)
- SW12 pad 1: /COL11 -> /KEY_MATRIX/COL2
- SW12 pad 2: Net-(D12-A) -> Net-(D13-A)
- SW13 pad 1: /COL12 -> /KEY_MATRIX/COL2
- SW13 pad 2: Net-(D13-A) -> Net-(D14-A)
- SW14 pad 1: /COL13 -> /KEY_MATRIX/COL3
- SW14 pad 2: Net-(D14-A) -> Net-(D15-A)
- SW15 pad 1: /COL14 -> /KEY_MATRIX/COL3
- SW15 pad 2: Net-(D15-A) -> Net-(D16-A)
- SW16 pad 1: /COL0 -> /KEY_MATRIX/COL3
- SW16 pad 2: Net-(D16-A) -> Net-(D17-A)
- SW17 pad 1: /COL1 -> /KEY_MATRIX/COL3
- SW17 pad 2: Net-(D17-A) -> Net-(D18-A)
- SW18 pad 1: /COL2 -> /KEY_MATRIX/COL3
- SW18 pad 2: Net-(D18-A) -> Net-(D19-A)
- SW19 pad 1: /COL3 -> /KEY_MATRIX/COL4
- SW19 pad 2: Net-(D19-A) -> Net-(D20-A)
- SW2 pad 1: /COL1 -> /KEY_MATRIX/COL0
- SW2 pad 2: Net-(D2-A) -> Net-(D3-A)
- SW20 pad 1: /COL4 -> /KEY_MATRIX/COL4
- SW20 pad 2: Net-(D20-A) -> Net-(D21-A)
- SW21 pad 1: /COL5 -> /KEY_MATRIX/COL4
- SW21 pad 2: Net-(D21-A) -> Net-(D22-A)
- SW22 pad 1: /COL7 -> /KEY_MATRIX/COL4
- SW22 pad 2: Net-(D22-A) -> Net-(D23-A)
- SW23 pad 1: /COL8 -> /KEY_MATRIX/COL4
- SW23 pad 2: Net-(D23-A) -> Net-(D24-A)
- SW24 pad 1: /COL9 -> /KEY_MATRIX/COL5
- SW24 pad 2: Net-(D24-A) -> Net-(D25-A)
- SW25 pad 1: /COL10 -> /KEY_MATRIX/COL5
- SW25 pad 2: Net-(D25-A) -> Net-(D26-A)
- SW26 pad 1: /COL11 -> /KEY_MATRIX/COL5
- SW26 pad 2: Net-(D26-A) -> Net-(D27-A)
- SW27 pad 1: /COL12 -> /KEY_MATRIX/COL5
- SW27 pad 2: Net-(D27-A) -> Net-(D28-A)
- SW28 pad 1: /COL13 -> /KEY_MATRIX/COL5
- SW28 pad 2: Net-(D28-A) -> Net-(D29-A)
- SW29 pad 1: /COL14 -> /KEY_MATRIX/COL6
- SW29 pad 2: Net-(D29-A) -> Net-(D30-A)
- SW3 pad 1: /COL2 -> /KEY_MATRIX/COL0
- SW3 pad 2: Net-(D3-A) -> Net-(D4-A)
- SW30 pad 1: /COL0 -> /KEY_MATRIX/COL7
- SW30 pad 2: Net-(D30-A) -> Net-(D31-A)
- SW31 pad 1: /COL1 -> /KEY_MATRIX/COL7
- SW31 pad 2: Net-(D31-A) -> Net-(D32-A)
- SW32 pad 1: /COL2 -> /KEY_MATRIX/COL7
- SW32 pad 2: Net-(D32-A) -> Net-(D33-A)
- SW33 pad 1: /COL3 -> /KEY_MATRIX/COL7
- SW33 pad 2: Net-(D33-A) -> Net-(D34-A)
- SW34 pad 1: /COL4 -> /KEY_MATRIX/COL7
- SW34 pad 2: Net-(D34-A) -> Net-(D35-A)
- SW35 pad 1: /COL5 -> /KEY_MATRIX/COL8
- SW35 pad 2: Net-(D35-A) -> Net-(D36-A)
- SW36 pad 1: /COL7 -> /KEY_MATRIX/COL8
- SW36 pad 2: Net-(D36-A) -> Net-(D37-A)
- SW37 pad 1: /COL8 -> /KEY_MATRIX/COL8
- SW37 pad 2: Net-(D37-A) -> Net-(D38-A)
- SW38 pad 1: /COL9 -> /KEY_MATRIX/COL8
- SW38 pad 2: Net-(D38-A) -> Net-(D39-A)
- SW39 pad 1: /COL10 -> /KEY_MATRIX/COL9
- SW39 pad 2: Net-(D39-A) -> Net-(D40-A)
- SW4 pad 1: /COL3 -> /KEY_MATRIX/COL0
- SW4 pad 2: Net-(D4-A) -> Net-(D5-A)
- SW40 pad 1: /COL12 -> /KEY_MATRIX/COL9
- SW40 pad 2: Net-(D40-A) -> Net-(D41-A)
- SW41 pad 1: /COL13 -> /KEY_MATRIX/COL9
- SW41 pad 2: Net-(D41-A) -> Net-(D42-A)
- SW42 pad 1: /COL14 -> /KEY_MATRIX/COL9
- SW42 pad 2: Net-(D42-A) -> Net-(D43-A)
- SW43 pad 1: /COL0 -> /KEY_MATRIX/COL9
- SW43 pad 2: Net-(D43-A) -> Net-(D44-A)
- SW44 pad 1: /COL1 -> /KEY_MATRIX/COL10
- SW44 pad 2: Net-(D44-A) -> Net-(D45-A)
- SW45 pad 1: /COL2 -> /KEY_MATRIX/COL10
- SW45 pad 2: Net-(D45-A) -> Net-(D46-A)
- SW46 pad 1: /COL3 -> /KEY_MATRIX/COL10
- SW46 pad 2: Net-(D46-A) -> Net-(D47-A)
- SW47 pad 1: /COL4 -> /KEY_MATRIX/COL10
- SW47 pad 2: Net-(D47-A) -> Net-(D48-A)
- SW48 pad 1: /COL5 -> /KEY_MATRIX/COL11
- SW48 pad 2: Net-(D48-A) -> Net-(D49-A)
- SW49 pad 1: /COL7 -> /KEY_MATRIX/COL11
- SW49 pad 2: Net-(D49-A) -> Net-(D50-A)
- SW5 pad 1: /COL4 -> /KEY_MATRIX/COL0
- SW5 pad 2: Net-(D5-A) -> Net-(D6-A)
- SW50 pad 1: /COL8 -> /KEY_MATRIX/COL12
- SW50 pad 2: Net-(D50-A) -> Net-(D51-A)
- SW51 pad 1: /COL9 -> /KEY_MATRIX/COL12
- SW51 pad 2: Net-(D51-A) -> Net-(D52-A)
- SW52 pad 1: /COL10 -> /KEY_MATRIX/COL12
- SW52 pad 2: Net-(D52-A) -> Net-(D53-A)
- SW53 pad 1: /COL12 -> /KEY_MATRIX/COL12
- SW53 pad 2: Net-(D53-A) -> Net-(D54-A)
- SW54 pad 1: /COL14 -> /KEY_MATRIX/COL13
- SW54 pad 2: Net-(D54-A) -> Net-(D55-A)
- SW55 pad 1: /COL0 -> /KEY_MATRIX/COL13
- SW55 pad 2: Net-(D55-A) -> Net-(D56-A)
- SW56 pad 1: /COL3 -> /KEY_MATRIX/COL13
- SW56 pad 2: Net-(D56-A) -> Net-(D57-A)
- SW57 pad 1: /COL4 -> /KEY_MATRIX/COL14
- SW57 pad 2: Net-(D57-A) -> Net-(D58-A)
- SW58 pad 1: /COL5 -> /KEY_MATRIX/COL14
- SW58 pad 2: Net-(D58-A) -> Net-(D59-A)
- SW59 pad 1: /COL7 -> /KEY_MATRIX/COL14
- SW59 pad 2: Net-(D59-A) -> Net-(D60-A)
- SW6 pad 1: /COL5 -> /KEY_MATRIX/COL1
- SW6 pad 2: Net-(D6-A) -> Net-(D7-A)
- SW60 pad 1: /COL9 -> /KEY_MATRIX/COL14
- SW60 pad 2: Net-(D60-A) -> Net-(D61-A)
- SW61 pad 1: /COL14 -> /KEY_MATRIX/COL14
- SW61 pad 2: Net-(D61-A) -> Net-(D62-A)
- SW7 pad 1: /COL6 -> /KEY_MATRIX/COL1
- SW7 pad 2: Net-(D7-A) -> Net-(D8-A)
- SW8 pad 1: /COL7 -> /KEY_MATRIX/COL1
- SW8 pad 2: Net-(D8-A) -> Net-(D9-A)
- SW9 pad 1: /COL8 -> /KEY_MATRIX/COL1
- SW9 pad 2: Net-(D9-A) -> Net-(D10-A)
Other:
- board outline added: 3.6 x 3.2 mm

Commit message: schematics done
Parts:
- added C1: 470u, Capacitor_Tantalum_SMD:CP_EIA-7343-31_Kemet-D_HandSolder, F.Cu at (141.6, 242.4)
- added C10: 100n, Capacitor_SMD:C_0603_1608Metric_Pad1.08x0.95mm_HandSolder, F.Cu at (108.2, 260.8)
- added C11: 100n, Capacitor_SMD:C_0603_1608Metric_Pad1.08x0.95mm_HandSolder, F.Cu at (112.5, 240.7)
- added C12: 100n, Capacitor_SMD:C_0603_1608Metric_Pad1.08x0.95mm_HandSolder, F.Cu at (112.5, 243.2)
- added C13: 100n, Capacitor_SMD:C_0603_1608Metric_Pad1.08x0.95mm_HandSolder, F.Cu at (112.5, 245.7)
- added C14: 100n, Capacitor_SMD:C_0603_1608Metric_Pad1.08x0.95mm_HandSolder, F.Cu at (112.5, 248.2)
- added C15: 100n, Capacitor_SMD:C_0603_1608Metric_Pad1.08x0.95mm_HandSolder, F.Cu at (112.5, 250.7)
- added C16: 100n, Capacitor_SMD:C_0603_1608Metric_Pad1.08x0.95mm_HandSolder, F.Cu at (112.5, 253.2)
- added C17: 100n, Capacitor_SMD:C_0603_1608Metric_Pad1.08x0.95mm_HandSolder, F.Cu at (112.5, 255.8)
- added C18: 100n, Capacitor_SMD:C_0603_1608Metric_Pad1.08x0.95mm_HandSolder, F.Cu at (112.5, 258.3)
- added C19: 100n, Capacitor_SMD:C_0603_1608Metric_Pad1.08x0.95mm_HandSolder, F.Cu at (112.5, 260.8)
- added C2: 100n, Capacitor_SMD:C_0603_1608Metric_Pad1.08x0.95mm_HandSolder, F.Cu at (108.2, 240.7)
- added C20: 100n, Capacitor_SMD:C_0603_1608Metric_Pad1.08x0.95mm_HandSolder, F.Cu at (116.9, 240.7)
- added C21: 100n, Capacitor_SMD:C_0603_1608Metric_Pad1.08x0.95mm_HandSolder, F.Cu at (116.9, 243.2)
- added C22: 100n, Capacitor_SMD:C_0603_1608Metric_Pad1.08x0.95mm_HandSolder, F.Cu at (116.9, 245.7)
- added C23: 100n, Capacitor_SMD:C_0603_1608Metric_Pad1.08x0.95mm_HandSolder, F.Cu at (116.9, 248.2)
- added C24: 100n, Capacitor_SMD:C_0603_1608Metric_Pad1.08x0.95mm_HandSolder, F.Cu at (116.9, 250.7)
- added C25: 100n, Capacitor_SMD:C_0603_1608Metric_Pad1.08x0.95mm_HandSolder, F.Cu at (116.9, 253.2)
- added C26: 100n, Capacitor_SMD:C_0603_1608Metric_Pad1.08x0.95mm_HandSolder, F.Cu at (116.9, 255.8)
- added C27: 100n, Capacitor_SMD:C_0603_1608Metric_Pad1.08x0.95mm_HandSolder, F.Cu at (116.9, 258.3)
- added C28: 100n, Capacitor_SMD:C_0603_1608Metric_Pad1.08x0.95mm_HandSolder, F.Cu at (116.9, 260.8)
- added C29: 100n, Capacitor_SMD:C_0603_1608Metric_Pad1.08x0.95mm_HandSolder, F.Cu at (121.2, 240.7)
- added C3: 100n, Capacitor_SMD:C_0603_1608Metric_Pad1.08x0.95mm_HandSolder, F.Cu at (108.2, 243.2)
- added C30: 100n, Capacitor_SMD:C_0603_1608Metric_Pad1.08x0.95mm_HandSolder, F.Cu at (121.2, 243.2)
- added C31: 100n, Capacitor_SMD:C_0603_1608Metric_Pad1.08x0.95mm_HandSolder, F.Cu at (121.2, 245.7)
- added C32: 100n, Capacitor_SMD:C_0603_1608Metric_Pad1.08x0.95mm_HandSolder, F.Cu at (121.2, 248.2)
- added C33: 100n, Capacitor_SMD:C_0603_1608Metric_Pad1.08x0.95mm_HandSolder, F.Cu at (121.2, 250.7)
- added C34: 100n, Capacitor_SMD:C_0603_1608Metric_Pad1.08x0.95mm_HandSolder, F.Cu at (121.2, 253.2)
- added C35: 100n, Capacitor_SMD:C_0603_1608Metric_Pad1.08x0.95mm_HandSolder, F.Cu at (121.2, 255.8)
- added C36: 100n, Capacitor_SMD:C_0603_1608Metric_Pad1.08x0.95mm_HandSolder, F.Cu at (121.2, 258.3)
- added C37: 100n, Capacitor_SMD:C_0603_1608Metric_Pad1.08x0.95mm_HandSolder, F.Cu at (121.2, 260.8)
- added C38: 100n, Capacitor_SMD:C_0603_1608Metric_Pad1.08x0.95mm_HandSolder, F.Cu at (125.6, 240.7)
- added C39: 100n, Capacitor_SMD:C_0603_1608Metric_Pad1.08x0.95mm_HandSolder, F.Cu at (125.6, 243.2)
- added C4: 100n, Capacitor_SMD:C_0603_1608Metric_Pad1.08x0.95mm_HandSolder, F.Cu at (108.2, 245.7)
- added C40: 100n, Capacitor_SMD:C_0603_1608Metric_Pad1.08x0.95mm_HandSolder, F.Cu at (125.6, 245.7)
- added C41: 100n, Capacitor_SMD:C_0603_1608Metric_Pad1.08x0.95mm_HandSolder, F.Cu at (125.6, 248.2)
- added C42: 100n, Capacitor_SMD:C_0603_1608Metric_Pad1.08x0.95mm_HandSolder, F.Cu at (125.6, 250.7)
- added C43: 100n, Capacitor_SMD:C_0603_1608Metric_Pad1.08x0.95mm_HandSolder, F.Cu at (125.6, 253.2)
- added C44: 100n, Capacitor_SMD:C_0603_1608Metric_Pad1.08x0.95mm_HandSolder, F.Cu at (125.6, 255.8)
- added C45: 100n, Capacitor_SMD:C_0603_1608Metric_Pad1.08x0.95mm_HandSolder, F.Cu at (125.6, 258.3)
- added C46: 100n, Capacitor_SMD:C_0603_1608Metric_Pad1.08x0.95mm_HandSolder, F.Cu at (125.6, 260.8)
- added C47: 100n, Capacitor_SMD:C_0603_1608Metric_Pad1.08x0.95mm_HandSolder, F.Cu at (129.9, 240.7)
- added C48: 100n, Capacitor_SMD:C_0603_1608Metric_Pad1.08x0.95mm_HandSolder, F.Cu at (129.9, 243.2)
- added C49: 100n, Capacitor_SMD:C_0603_1608Metric_Pad1.08x0.95mm_HandSolder, F.Cu at (129.9, 245.7)
- added C5: 100n, Capacitor_SMD:C_0603_1608Metric_Pad1.08x0.95mm_HandSolder, F.Cu at (108.2, 248.2)
- added C50: 100n, Capacitor_SMD:C_0603_1608Metric_Pad1.08x0.95mm_HandSolder, F.Cu at (129.9, 248.2)
- added C51: 100n, Capacitor_SMD:C_0603_1608Metric_Pad1.08x0.95mm_HandSolder, F.Cu at (129.9, 250.7)
- added C52: 100n, Capacitor_SMD:C_0603_1608Metric_Pad1.08x0.95mm_HandSolder, F.Cu at (129.9, 253.2)
- added C53: 100n, Capacitor_SMD:C_0603_1608Metric_Pad1.08x0.95mm_HandSolder, F.Cu at (129.9, 255.8)
- added C54: 100n, Capacitor_SMD:C_0603_1608Metric_Pad1.08x0.95mm_HandSolder, F.Cu at (129.9, 258.3)
- added C55: 100n, Capacitor_SMD:C_0603_1608Metric_Pad1.08x0.95mm_HandSolder, F.Cu at (129.9, 260.8)
- added C56: 100n, Capacitor_SMD:C_0603_1608Metric_Pad1.08x0.95mm_HandSolder, F.Cu at (134.3, 240.7)
- added C57: 100n, Capacitor_SMD:C_0603_1608Metric_Pad1.08x0.95mm_HandSolder, F.Cu at (134.3, 243.2)
- added C58: 100n, Capacitor_SMD:C_0603_1608Metric_Pad1.08x0.95mm_HandSolder, F.Cu at (134.3, 245.7)
- added C59: 100n, Capacitor_SMD:C_0603_1608Metric_Pad1.08x0.95mm_HandSolder, F.Cu at (134.3, 248.2)
- added C6: 100n, Capacitor_SMD:C_0603_1608Metric_Pad1.08x0.95mm_HandSolder, F.Cu at (108.2, 250.7)
- added C60: 100n, Capacitor_SMD:C_0603_1608Metric_Pad1.08x0.95mm_HandSolder, F.Cu at (134.3, 250.7)
- added C61: 100n, Capacitor_SMD:C_0603_1608Metric_Pad1.08x0.95mm_HandSolder, F.Cu at (134.3, 253.2)
- added C62: 100n, Capacitor_SMD:C_0603_1608Metric_Pad1.08x0.95mm_HandSolder, F.Cu at (134.3, 255.8)
- added C7: 100n, Capacitor_SMD:C_0603_1608Metric_Pad1.08x0.95mm_HandSolder, F.Cu at (108.2, 253.2)
- added C8: 100n, Capacitor_SMD:C_0603_1608Metric_Pad1.08x0.95mm_HandSolder, F.Cu at (108.2, 255.8)
- added C9: 100n, Capacitor_SMD:C_0603_1608Metric_Pad1.08x0.95mm_HandSolder, F.Cu at (108.2, 258.3)
- added D100: SK6812MINI-E, LED_SMD:LED_SK6812MINI-E_3.2x2.8mm_P1.5mm_ReverseMount, F.Cu at (143.9, 207.8)
- added D101: SK6812MINI-E, LED_SMD:LED_SK6812MINI-E_3.2x2.8mm_P1.5mm_ReverseMount, F.Cu at (143.9, 212.7)
- added D102: SK6812MINI-E, LED_SMD:LED_SK6812MINI-E_3.2x2.8mm_P1.5mm_ReverseMount, F.Cu at (143.9, 217.5)
- added D103: SK6812MINI-E, LED_SMD:LED_SK6812MINI-E_3.2x2.8mm_P1.5mm_ReverseMount, F.Cu at (143.9, 222.4)
- added D104: SK6812MINI-E, LED_SMD:LED_SK6812MINI-E_3.2x2.8mm_P1.5mm_ReverseMount, F.Cu at (143.9, 227.3)
- added D105: SK6812MINI-E, LED_SMD:LED_SK6812MINI-E_3.2x2.8mm_P1.5mm_ReverseMount, F.Cu at (143.9, 232.1)
- added D106: SK6812MINI-E, LED_SMD:LED_SK6812MINI-E_3.2x2.8mm_P1.5mm_ReverseMount, F.Cu at (143.9, 237.0)
- added D107: SK6812MINI-E, LED_SMD:LED_SK6812MINI-E_3.2x2.8mm_P1.5mm_ReverseMount, F.Cu at (152.3, 198.0)
- added D108: SK6812MINI-E, LED_SMD:LED_SK6812MINI-E_3.2x2.8mm_P1.5mm_ReverseMount, F.Cu at (152.3, 202.9)
- added D109: SK6812MINI-E, LED_SMD:LED_SK6812MINI-E_3.2x2.8mm_P1.5mm_ReverseMount, F.Cu at (152.3, 207.8)
- added D110: SK6812MINI-E, LED_SMD:LED_SK6812MINI-E_3.2x2.8mm_P1.5mm_ReverseMount, F.Cu at (152.3, 212.7)
- added D111: SK6812MINI-E, LED_SMD:LED_SK6812MINI-E_3.2x2.8mm_P1.5mm_ReverseMount, F.Cu at (152.3, 217.5)
- added D112: SK6812MINI-E, LED_SMD:LED_SK6812MINI-E_3.2x2.8mm_P1.5mm_ReverseMount, F.Cu at (152.3, 222.4)
- added D113: SK6812MINI-E, LED_SMD:LED_SK6812MINI-E_3.2x2.8mm_P1.5mm_ReverseMount, F.Cu at (152.3, 227.3)
- added D114: SK6812MINI-E, LED_SMD:LED_SK6812MINI-E_3.2x2.8mm_P1.5mm_ReverseMount, F.Cu at (152.3, 232.1)
- added D115: SK6812MINI-E, LED_SMD:LED_SK6812MINI-E_3.2x2.8mm_P1.5mm_ReverseMount, F.Cu at (152.3, 237.0)
- added D116: SK6812MINI-E, LED_SMD:LED_SK6812MINI-E_3.2x2.8mm_P1.5mm_ReverseMount, F.Cu at (160.7, 198.0)
- added D117: SK6812MINI-E, LED_SMD:LED_SK6812MINI-E_3.2x2.8mm_P1.5mm_ReverseMount, F.Cu at (160.7, 202.9)
- added D118: SK6812MINI-E, LED_SMD:LED_SK6812MINI-E_3.2x2.8mm_P1.5mm_ReverseMount, F.Cu at (160.7, 207.8)
- added D119: SK6812MINI-E, LED_SMD:LED_SK6812MINI-E_3.2x2.8mm_P1.5mm_ReverseMount, F.Cu at (160.7, 212.7)
- added D120: SK6812MINI-E, LED_SMD:LED_SK6812MINI-E_3.2x2.8mm_P1.5mm_ReverseMount, F.Cu at (160.7, 217.5)
- added D121: SK6812MINI-E, LED_SMD:LED_SK6812MINI-E_3.2x2.8mm_P1.5mm_ReverseMount, F.Cu at (160.7, 222.4)
- added D122: SK6812MINI-E, LED_SMD:LED_SK6812MINI-E_3.2x2.8mm_P1.5mm_ReverseMount, F.Cu at (160.7, 227.3)
- added D63: SK6812MINI-E, LED_SMD:LED_SK6812MINI-E_3.2x2.8mm_P1.5mm_ReverseMount, F.Cu at (110.2, 202.9)
- added D64: SK6812MINI-E, LED_SMD:LED_SK6812MINI-E_3.2x2.8mm_P1.5mm_ReverseMount, F.Cu at (110.2, 207.8)
- added D65: SK6812MINI-E, LED_SMD:LED_SK6812MINI-E_3.2x2.8mm_P1.5mm_ReverseMount, F.Cu at (110.2, 212.7)
- added D66: SK6812MINI-E, LED_SMD:LED_SK6812MINI-E_3.2x2.8mm_P1.5mm_ReverseMount, F.Cu at (110.2, 217.5)
- added D67: SK6812MINI-E, LED_SMD:LED_SK6812MINI-E_3.2x2.8mm_P1.5mm_ReverseMount, F.Cu at (110.2, 222.4)
- added D68: SK6812MINI-E, LED_SMD:LED_SK6812MINI-E_3.2x2.8mm_P1.5mm_ReverseMount, F.Cu at (110.2, 227.3)
- added D69: SK6812MINI-E, LED_SMD:LED_SK6812MINI-E_3.2x2.8mm_P1.5mm_ReverseMount, F.Cu at (110.2, 232.1)
- added D70: SK6812MINI-E, LED_SMD:LED_SK6812MINI-E_3.2x2.8mm_P1.5mm_ReverseMount, F.Cu at (110.2, 237.0)
- added D71: SK6812MINI-E, LED_SMD:LED_SK6812MINI-E_3.2x2.8mm_P1.5mm_ReverseMount, F.Cu at (118.6, 198.0)
- added D72: SK6812MINI-E, LED_SMD:LED_SK6812MINI-E_3.2x2.8mm_P1.5mm_ReverseMount, F.Cu at (118.6, 202.9)
- added D73: SK6812MINI-E, LED_SMD:LED_SK6812MINI-E_3.2x2.8mm_P1.5mm_ReverseMount, F.Cu at (118.6, 207.8)
- added D74: SK6812MINI-E, LED_SMD:LED_SK6812MINI-E_3.2x2.8mm_P1.5mm_ReverseMount, F.Cu at (118.6, 212.7)
- added D75: SK6812MINI-E, LED_SMD:LED_SK6812MINI-E_3.2x2.8mm_P1.5mm_ReverseMount, F.Cu at (118.6, 217.5)
- added D76: SK6812MINI-E, LED_SMD:LED_SK6812MINI-E_3.2x2.8mm_P1.5mm_ReverseMount, F.Cu at (118.6, 222.4)
- added D77: SK6812MINI-E, LED_SMD:LED_SK6812MINI-E_3.2x2.8mm_P1.5mm_ReverseMount, F.Cu at (118.6, 227.3)
- added D78: SK6812MINI-E, LED_SMD:LED_SK6812MINI-E_3.2x2.8mm_P1.5mm_ReverseMount, F.Cu at (118.6, 232.1)
- added D79: SK6812MINI-E, LED_SMD:LED_SK6812MINI-E_3.2x2.8mm_P1.5mm_ReverseMount, F.Cu at (118.6, 237.0)
- added D80: SK6812MINI-E, LED_SMD:LED_SK6812MINI-E_3.2x2.8mm_P1.5mm_ReverseMount, F.Cu at (127.0, 198.0)
- added D81: SK6812MINI-E, LED_SMD:LED_SK6812MINI-E_3.2x2.8mm_P1.5mm_ReverseMount, F.Cu at (127.0, 202.9)
- added D82: SK6812MINI-E, LED_SMD:LED_SK6812MINI-E_3.2x2.8mm_P1.5mm_ReverseMount, F.Cu at (127.0, 207.8)
- added D83: SK6812MINI-E, LED_SMD:LED_SK6812MINI-E_3.2x2.8mm_P1.5mm_ReverseMount, F.Cu at (127.0, 212.7)
- added D84: SK6812MINI-E, LED_SMD:LED_SK6812MINI-E_3.2x2.8mm_P1.5mm_ReverseMount, F.Cu at (127.0, 217.5)
- added D85: SK6812MINI-E, LED_SMD:LED_SK6812MINI-E_3.2x2.8mm_P1.5mm_ReverseMount, F.Cu at (127.0, 222.4)
- added D86: SK6812MINI-E, LED_SMD:LED_SK6812MINI-E_3.2x2.8mm_P1.5mm_ReverseMount, F.Cu at (127.0, 227.3)
- added D87: SK6812MINI-E, LED_SMD:LED_SK6812MINI-E_3.2x2.8mm_P1.5mm_ReverseMount, F.Cu at (127.0, 232.1)
- added D88: SK6812MINI-E, LED_SMD:LED_SK6812MINI-E_3.2x2.8mm_P1.5mm_ReverseMount, F.Cu at (127.0, 237.0)
- added D89: SK6812MINI-E, LED_SMD:LED_SK6812MINI-E_3.2x2.8mm_P1.5mm_ReverseMount, F.Cu at (135.5, 198.0)
- added D90: SK6812MINI-E, LED_SMD:LED_SK6812MINI-E_3.2x2.8mm_P1.5mm_ReverseMount, F.Cu at (135.5, 202.9)
- added D91: SK6812MINI-E, LED_SMD:LED_SK6812MINI-E_3.2x2.8mm_P1.5mm_ReverseMount, F.Cu at (135.5, 207.8)
- added D92: SK6812MINI-E, LED_SMD:LED_SK6812MINI-E_3.2x2.8mm_P1.5mm_ReverseMount, F.Cu at (135.5, 212.7)
- added D93: SK6812MINI-E, LED_SMD:LED_SK6812MINI-E_3.2x2.8mm_P1.5mm_ReverseMount, F.Cu at (135.5, 217.5)
- added D94: SK6812MINI-E, LED_SMD:LED_SK6812MINI-E_3.2x2.8mm_P1.5mm_ReverseMount, F.Cu at (135.5, 222.4)
- added D95: SK6812MINI-E, LED_SMD:LED_SK6812MINI-E_3.2x2.8mm_P1.5mm_ReverseMount, F.Cu at (135.5, 227.3)
- added D96: SK6812MINI-E, LED_SMD:LED_SK6812MINI-E_3.2x2.8mm_P1.5mm_ReverseMount, F.Cu at (135.5, 232.1)
- added D97: SK6812MINI-E, LED_SMD:LED_SK6812MINI-E_3.2x2.8mm_P1.5mm_ReverseMount, F.Cu at (135.5, 237.0)
- added D98: SK6812MINI-E, LED_SMD:LED_SK6812MINI-E_3.2x2.8mm_P1.5mm_ReverseMount, F.Cu at (143.9, 198.0)
- added D99: SK6812MINI-E, LED_SMD:LED_SK6812MINI-E_3.2x2.8mm_P1.5mm_ReverseMount, F.Cu at (143.9, 202.9)
- added H1: MountingHole, Capacitor_Tantalum_SMD:CP_EIA-7343-31_Kemet-D_HandSolder, F.Cu at (311.2, 88.7)
- added H2: MountingHole, MountingHole:MountingHole_3.2mm_M3, F.Cu at (310.0, 50.0)
- added H3: MountingHole, MountingHole:MountingHole_3.2mm_M3, F.Cu at (310.0, 57.9)
- added H4: MountingHole, MountingHole:MountingHole_3.2mm_M3, F.Cu at (310.0, 65.9)
- added H5: MountingHole, MountingHole:MountingHole_3.2mm_M3, F.Cu at (310.0, 73.8)
- added H6: MountingHole, MountingHole:MountingHole_3.2mm_M3, F.Cu at (310.0, 81.8)
- added R1: 330, Resistor_SMD:R_0603_1608Metric_Pad0.98x0.95mm_HandSolder, F.Cu at (134.3, 258.3)
- D1: value SK6812MINI-E -> 1N4148; footprint LED_SMD:LED_SK6812MINI-E_3.2x2.8mm_P1.5mm_ReverseMount -> Diode_THT:D_DO-35_SOD27_P7.62mm_Horizontal
- D62: value 1N4148 -> SK6812MINI-E; footprint Diode_THT:D_DO-35_SOD27_P7.62mm_Horizontal -> LED_SMD:LED_SK6812MINI-E_3.2x2.8mm_P1.5mm_ReverseMount
- SW1, SW10, SW11, SW12, SW13, SW14, SW15, SW16, SW17, SW18, SW19, SW2, SW20, SW21, SW22, SW23, SW24, SW25, SW26, SW27, SW28, SW29, SW3, SW30, SW31, SW32, SW33, SW34, SW35, SW36, SW37, SW38, SW39, SW4, SW40, SW41, SW42, SW43, SW44, SW45, SW46, SW47, SW48, SW49, SW5, SW50, SW51, SW52, SW53, SW54, SW55, SW56, SW57, SW58, SW59, SW6, SW60, SW61, SW7, SW8, SW9: footprint PCM_marbastlib-mx:SW_MX_1u -> PCM_marbastlib-mx:SW_MX_HS_CPG151101S11_1u
- moved D62 140.3 mm to (110.2, 198.0)
- moved D1 83.5 mm to (227.6, 128.9)
- moved D14 73.9 mm to (238.4, 128.9)
- moved D27 73.9 mm to (249.2, 128.9)
- moved D40 73.9 mm to (259.9, 128.9)
- moved D53 73.9 mm to (270.7, 128.9)
- moved S5 32.0 mm to (240.5, 116.4)
- moved S2 32.0 mm to (240.5, 55.5)
- moved S3 32.0 mm to (240.5, 75.8)
- moved S4 32.0 mm to (240.5, 96.1)
- moved A1 32.0 mm to (285.1, 69.6)
- moved S1 32.0 mm to (247.7, 182.9)
- moved SW55 30.9 mm to (216.8, 53.5)
- moved SW56 30.9 mm to (216.8, 68.6)
- moved SW57 30.9 mm to (216.8, 83.6)
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Connections:
- A1 pad 40: unconnected-(A1-VBUS-Pad40) -> +5V
- D1 pad 1: unconnected-(D1-VSS-Pad1) -> /ROW0
- D1 pad 2: unconnected-(D1-DIN-Pad2) -> Net-(D1-A)
- D10 pad 1: /KEY_MATRIX/ROW3 -> /ROW0
- D11 pad 1: /KEY_MATRIX/ROW0 -> /ROW0
- D12 pad 1: /KEY_MATRIX/ROW1 -> /ROW0
- D13 pad 1: /KEY_MATRIX/ROW2 -> /ROW0
- D14 pad 1: /KEY_MATRIX/ROW3 -> /ROW0
- D15 pad 1: /KEY_MATRIX/ROW0 -> /ROW0
- D16 pad 1: /KEY_MATRIX/ROW1 -> /ROW1
- D17 pad 1: /KEY_MATRIX/ROW2 -> /ROW1
- D18 pad 1: /KEY_MATRIX/ROW3 -> /ROW1
- D19 pad 1: /KEY_MATRIX/ROW4 -> /ROW1
- D2 pad 1: /KEY_MATRIX/ROW0 -> /ROW0
- D20 pad 1: /KEY_MATRIX/ROW0 -> /ROW1
- D21 pad 1: /KEY_MATRIX/ROW1 -> /ROW1
- D22 pad 1: /KEY_MATRIX/ROW2 -> /ROW1
- D23 pad 1: /KEY_MATRIX/ROW3 -> /ROW1
- D24 pad 1: /KEY_MATRIX/ROW4 -> /ROW1
- D25 pad 1: /KEY_MATRIX/ROW0 -> /ROW1
- D26 pad 1: /KEY_MATRIX/ROW1 -> /ROW1
- D27 pad 1: /KEY_MATRIX/ROW2 -> /ROW1
- D28 pad 1: /KEY_MATRIX/ROW3 -> /ROW1
- D29 pad 1: /KEY_MATRIX/ROW4 -> /ROW1
- D3 pad 1: /KEY_MATRIX/ROW1 -> /ROW0
- D30 pad 1: /KEY_MATRIX/ROW0 -> /ROW2
- D31 pad 1: /KEY_MATRIX/ROW0 -> /ROW2
- D32 pad 1: /KEY_MATRIX/ROW1 -> /ROW2
- D33 pad 1: /KEY_MATRIX/ROW2 -> /ROW2
- D34 pad 1: /KEY_MATRIX/ROW3 -> /ROW2
- D35 pad 1: /KEY_MATRIX/ROW4 -> /ROW2
- D36 pad 1: /KEY_MATRIX/ROW0 -> /ROW2
- D37 pad 1: /KEY_MATRIX/ROW1 -> /ROW2
- D38 pad 1: /KEY_MATRIX/ROW2 -> /ROW2
- D39 pad 1: /KEY_MATRIX/ROW3 -> /ROW2
- D4 pad 1: /KEY_MATRIX/ROW2 -> /ROW0
- D40 pad 1: /KEY_MATRIX/ROW0 -> /ROW2
- D41 pad 1: /KEY_MATRIX/ROW1 -> /ROW2
- D42 pad 1: /KEY_MATRIX/ROW2 -> /ROW2
- D43 pad 1: /KEY_MATRIX/ROW3 -> /ROW3
- D44 pad 1: /KEY_MATRIX/ROW4 -> /ROW3
- D45 pad 1: /KEY_MATRIX/ROW0 -> /ROW3
- D46 pad 1: /KEY_MATRIX/ROW1 -> /ROW3
- D47 pad 1: /KEY_MATRIX/ROW2 -> /ROW3
- D48 pad 1: /KEY_MATRIX/ROW3 -> /ROW3
- D49 pad 1: /KEY_MATRIX/ROW0 -> /ROW3
- D5 pad 1: /KEY_MATRIX/ROW3 -> /ROW0
- D50 pad 1: /KEY_MATRIX/ROW1 -> /ROW3
- D51 pad 1: /KEY_MATRIX/ROW0 -> /ROW3
- D52 pad 1: /KEY_MATRIX/ROW1 -> /ROW3
- D53 pad 1: /KEY_MATRIX/ROW2 -> /ROW3
- D54 pad 1: /KEY_MATRIX/ROW3 -> /ROW3
- D55 pad 1: /KEY_MATRIX/ROW0 -> /ROW4
- D56 pad 1: /KEY_MATRIX/ROW1 -> /ROW4
- D57 pad 1: /KEY_MATRIX/ROW2 -> /ROW4
- D58 pad 1: /KEY_MATRIX/ROW0 -> /ROW4
- D59 pad 1: /KEY_MATRIX/ROW1 -> /ROW4
- D6 pad 1: /KEY_MATRIX/ROW4 -> /ROW0
- D60 pad 1: /KEY_MATRIX/ROW2 -> /ROW4
- D61 pad 1: /KEY_MATRIX/ROW3 -> /ROW4
- D62 pad 1: /KEY_MATRIX/ROW4 -> GND
- D62 pad 2: Net-(D62-A) -> Net-(D62-DIN)
- D7 pad 1: /KEY_MATRIX/ROW0 -> /ROW0
- D8 pad 1: /KEY_MATRIX/ROW1 -> /ROW0
- D9 pad 1: /KEY_MATRIX/ROW2 -> /ROW0
- SW1 pad 1: /KEY_MATRIX/COL0 -> /COL0
- SW1 pad 2: Net-(D2-A) -> Net-(D1-A)
- SW10 pad 1: /KEY_MATRIX/COL2 -> /COL9
- SW10 pad 2: Net-(D11-A) -> Net-(D10-A)
- SW11 pad 1: /KEY_MATRIX/COL2 -> /COL10
- SW11 pad 2: Net-(D12-A) -> Net-(D11-A)
- SW12 pad 1: /KEY_MATRIX/COL2 -> /COL11
- SW12 pad 2: Net-(D13-A) -> Net-(D12-A)
- SW13 pad 1: /KEY_MATRIX/COL2 -> /COL12
- SW13 pad 2: Net-(D14-A) -> Net-(D13-A)
- SW14 pad 1: /KEY_MATRIX/COL3 -> /COL13
- SW14 pad 2: Net-(D15-A) -> Net-(D14-A)
- SW15 pad 1: /KEY_MATRIX/COL3 -> /COL14
- SW15 pad 2: Net-(D16-A) -> Net-(D15-A)
- SW16 pad 1: /KEY_MATRIX/COL3 -> /COL0
- SW16 pad 2: Net-(D17-A) -> Net-(D16-A)
- SW17 pad 1: /KEY_MATRIX/COL3 -> /COL1
- SW17 pad 2: Net-(D18-A) -> Net-(D17-A)
- SW18 pad 1: /KEY_MATRIX/COL3 -> /COL2
- SW18 pad 2: Net-(D19-A) -> Net-(D18-A)
- SW19 pad 1: /KEY_MATRIX/COL4 -> /COL3
- SW19 pad 2: Net-(D20-A) -> Net-(D19-A)
- SW2 pad 1: /KEY_MATRIX/COL0 -> /COL1
- SW2 pad 2: Net-(D3-A) -> Net-(D2-A)
- SW20 pad 1: /KEY_MATRIX/COL4 -> /COL4
- SW20 pad 2: Net-(D21-A) -> Net-(D20-A)
- SW21 pad 1: /KEY_MATRIX/COL4 -> /COL5
- SW21 pad 2: Net-(D22-A) -> Net-(D21-A)
- SW22 pad 1: /KEY_MATRIX/COL4 -> /COL7
- SW22 pad 2: Net-(D23-A) -> Net-(D22-A)
- SW23 pad 1: /KEY_MATRIX/COL4 -> /COL8
- SW23 pad 2: Net-(D24-A) -> Net-(D23-A)
- SW24 pad 1: /KEY_MATRIX/COL5 -> /COL9
- SW24 pad 2: Net-(D25-A) -> Net-(D24-A)
- SW25 pad 1: /KEY_MATRIX/COL5 -> /COL10
- SW25 pad 2: Net-(D26-A) -> Net-(D25-A)
- SW26 pad 1: /KEY_MATRIX/COL5 -> /COL11
- SW26 pad 2: Net-(D27-A) -> Net-(D26-A)
- SW27 pad 1: /KEY_MATRIX/COL5 -> /COL12
- SW27 pad 2: Net-(D28-A) -> Net-(D27-A)
- SW28 pad 1: /KEY_MATRIX/COL5 -> /COL13
- SW28 pad 2: Net-(D29-A) -> Net-(D28-A)
- SW29 pad 1: /KEY_MATRIX/COL6 -> /COL14
- SW29 pad 2: Net-(D30-A) -> Net-(D29-A)
- SW3 pad 1: /KEY_MATRIX/COL0 -> /COL2
- SW3 pad 2: Net-(D4-A) -> Net-(D3-A)
- SW30 pad 1: /KEY_MATRIX/COL7 -> /COL0
- SW30 pad 2: Net-(D31-A) -> Net-(D30-A)
- SW31 pad 1: /KEY_MATRIX/COL7 -> /COL1
- SW31 pad 2: Net-(D32-A) -> Net-(D31-A)
- SW32 pad 1: /KEY_MATRIX/COL7 -> /COL2
- SW32 pad 2: Net-(D33-A) -> Net-(D32-A)
- SW33 pad 1: /KEY_MATRIX/COL7 -> /COL3
- SW33 pad 2: Net-(D34-A) -> Net-(D33-A)
- SW34 pad 1: /KEY_MATRIX/COL7 -> /COL4
- SW34 pad 2: Net-(D35-A) -> Net-(D34-A)
- SW35 pad 1: /KEY_MATRIX/COL8 -> /COL5
- SW35 pad 2: Net-(D36-A) -> Net-(D35-A)
- SW36 pad 1: /KEY_MATRIX/COL8 -> /COL7
- SW36 pad 2: Net-(D37-A) -> Net-(D36-A)
- SW37 pad 1: /KEY_MATRIX/COL8 -> /COL8
- SW37 pad 2: Net-(D38-A) -> Net-(D37-A)
- SW38 pad 1: /KEY_MATRIX/COL8 -> /COL9
- SW38 pad 2: Net-(D39-A) -> Net-(D38-A)
- SW39 pad 1: /KEY_MATRIX/COL9 -> /COL10
- SW39 pad 2: Net-(D40-A) -> Net-(D39-A)
- SW4 pad 1: /KEY_MATRIX/COL0 -> /COL3
- SW4 pad 2: Net-(D5-A) -> Net-(D4-A)
- SW40 pad 1: /KEY_MATRIX/COL9 -> /COL12
- SW40 pad 2: Net-(D41-A) -> Net-(D40-A)
- SW41 pad 1: /KEY_MATRIX/COL9 -> /COL13
- SW41 pad 2: Net-(D42-A) -> Net-(D41-A)
- SW42 pad 1: /KEY_MATRIX/COL9 -> /COL14
- SW42 pad 2: Net-(D43-A) -> Net-(D42-A)
- SW43 pad 1: /KEY_MATRIX/COL9 -> /COL0
- SW43 pad 2: Net-(D44-A) -> Net-(D43-A)
- SW44 pad 1: /KEY_MATRIX/COL10 -> /COL1
- SW44 pad 2: Net-(D45-A) -> Net-(D44-A)
- SW45 pad 1: /KEY_MATRIX/COL10 -> /COL2
- SW45 pad 2: Net-(D46-A) -> Net-(D45-A)
- SW46 pad 1: /KEY_MATRIX/COL10 -> /COL3
- SW46 pad 2: Net-(D47-A) -> Net-(D46-A)
- SW47 pad 1: /KEY_MATRIX/COL10 -> /COL4
- SW47 pad 2: Net-(D48-A) -> Net-(D47-A)
- SW48 pad 1: /KEY_MATRIX/COL11 -> /COL5
- SW48 pad 2: Net-(D49-A) -> Net-(D48-A)
- SW49 pad 1: /KEY_MATRIX/COL11 -> /COL7
- SW49 pad 2: Net-(D50-A) -> Net-(D49-A)
- SW5 pad 1: /KEY_MATRIX/COL0 -> /COL4
- SW5 pad 2: Net-(D6-A) -> Net-(D5-A)
- SW50 pad 1: /KEY_MATRIX/COL12 -> /COL8
- SW50 pad 2: Net-(D51-A) -> Net-(D50-A)
- SW51 pad 1: /KEY_MATRIX/COL12 -> /COL9
- SW51 pad 2: Net-(D52-A) -> Net-(D51-A)
- SW52 pad 1: /KEY_MATRIX/COL12 -> /COL10
- SW52 pad 2: Net-(D53-A) -> Net-(D52-A)
- SW53 pad 1: /KEY_MATRIX/COL12 -> /COL12
- SW53 pad 2: Net-(D54-A) -> Net-(D53-A)
- SW54 pad 1: /KEY_MATRIX/COL13 -> /COL14
- SW54 pad 2: Net-(D55-A) -> Net-(D54-A)
- SW55 pad 1: /KEY_MATRIX/COL13 -> /COL0
- SW55 pad 2: Net-(D56-A) -> Net-(D55-A)
- SW56 pad 1: /KEY_MATRIX/COL13 -> /COL3
- SW56 pad 2: Net-(D57-A) -> Net-(D56-A)
- SW57 pad 1: /KEY_MATRIX/COL14 -> /COL4
- SW57 pad 2: Net-(D58-A) -> Net-(D57-A)
- SW58 pad 1: /KEY_MATRIX/COL14 -> /COL5
- SW58 pad 2: Net-(D59-A) -> Net-(D58-A)
- SW59 pad 1: /KEY_MATRIX/COL14 -> /COL7
- SW59 pad 2: Net-(D60-A) -> Net-(D59-A)
- SW6 pad 1: /KEY_MATRIX/COL1 -> /COL5
- SW6 pad 2: Net-(D7-A) -> Net-(D6-A)
- SW60 pad 1: /KEY_MATRIX/COL14 -> /COL9
- SW60 pad 2: Net-(D61-A) -> Net-(D60-A)
- SW61 pad 1: /KEY_MATRIX/COL14 -> /COL14
- SW61 pad 2: Net-(D62-A) -> Net-(D61-A)
- SW7 pad 1: /KEY_MATRIX/COL1 -> /COL6
- SW7 pad 2: Net-(D8-A) -> Net-(D7-A)
- SW8 pad 1: /KEY_MATRIX/COL1 -> /COL7
- SW8 pad 2: Net-(D9-A) -> Net-(D8-A)
- SW9 pad 1: /KEY_MATRIX/COL1 -> /COL8
- SW9 pad 2: Net-(D10-A) -> Net-(D9-A)

Commit message: pcb switch and diode placed but not rgbs
Parts:
- removed the C10 at (108.2, 260.8)
- removed the C11 at (112.5, 240.7)
- removed the C13 at (112.5, 245.7)
- removed C14, C15, C16, C18, C19, C20, C21, C23, C24, C25, C26, C28, C29, C30, C31, C33, C34, C35, C36, C38, C39, C40, C41, C43, C44, C45, C46, C48, C49, C50, C51, C53, C54, C55, C56, C58, C59, C60, C61, C62: 100n, Capacitor_SMD:C_0603_1608Metric_Pad1.08x0.95mm_HandSolder
- removed the C3 at (108.2, 243.2)
- removed the C4 at (108.2, 245.7)
- removed the C5 at (108.2, 248.2)
- removed the C6 at (108.2, 250.7)
- removed the C8 at (108.2, 255.8)
- removed the C9 at (108.2, 258.3)
- SW1, SW10, SW11, SW12, SW13, SW14, SW15, SW16, SW17, SW18, SW19, SW2, SW20, SW21, SW22, SW23, SW24, SW25, SW26, SW27, SW28, SW29, SW3, SW30, SW31, SW32, SW33, SW34, SW35, SW36, SW37, SW38, SW39, SW4, SW40, SW41, SW42, SW43, SW44, SW45, SW46, SW47, SW48, SW49, SW5, SW50, SW51, SW52, SW53, SW54, SW55, SW56, SW57, SW58, SW59, SW6, SW60, SW61, SW7, SW8, SW9: moved to B.Cu
- moved C1 341.1 mm to (480.9, 278.1)
- moved C5 341.1 mm to (451.8, 291.4)
- moved C8 341.1 mm to (460.5, 283.9)
- moved C9 341.1 mm to (460.5, 296.5)
- moved R1 341.1 mm to (473.5, 293.9)
- moved C10 341.1 mm to (464.8, 286.4)
- moved C11 341.1 mm to (469.2, 276.4)
- moved C12 341.1 mm to (469.2, 288.9)
- moved C13 341.1 mm to (473.5, 278.9)
- moved C2 341.1 mm to (447.4, 276.4)
- moved C3 341.1 mm to (447.4, 288.9)
- moved C4 341.1 mm to (451.8, 278.9)
- moved C7 341.1 mm to (456.1, 293.9)
- moved C6 341.1 mm to (456.1, 281.4)
- moved D63 332.9 mm to (442.5, 223.9)
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- renumbered C42 to C10, C47 to C11, C52 to C12, C57 to C13, C7 to C3, C12 to C4, C17 to C5, C22 to C6, C27 to C7, C32 to C8, C37 to C9
Other:
- board size 3.6 x 3.2 mm -> 341.2 x 141.6 mm

Commit message: placed rgbs and relative comps in pcb
Parts:
- H1: footprint Capacitor_Tantalum_SMD:CP_EIA-7343-31_Kemet-D_HandSolder -> MountingHole:MountingHole_3.2mm_M3
- RGB1: renamed from D62; moved to B.Cu
- RGB10: renamed from D71; moved to B.Cu
- RGB11: renamed from D72; moved to B.Cu
- RGB12: renamed from D73; moved to B.Cu
- RGB13: renamed from D74; moved to B.Cu
- RGB14: renamed from D75; moved to B.Cu
- RGB15: renamed from D76; moved to B.Cu
- RGB16: renamed from D77; moved to B.Cu
- RGB17: renamed from D78; moved to B.Cu
- RGB18: renamed from D79; moved to B.Cu
- RGB19: renamed from D80; moved to B.Cu
- RGB2: renamed from D63; moved to B.Cu
- RGB20: renamed from D81; moved to B.Cu
- RGB21: renamed from D82; moved to B.Cu
- RGB22: renamed from D83; moved to B.Cu
- RGB23: renamed from D84; moved to B.Cu
- RGB24: renamed from D85; moved to B.Cu
- RGB25: renamed from D86; moved to B.Cu
- RGB26: renamed from D87; moved to B.Cu
- RGB27: renamed from D88; moved to B.Cu
- RGB28: renamed from D89; moved to B.Cu
- RGB29: renamed from D90; moved to B.Cu
- RGB3: renamed from D64; moved to B.Cu
- RGB30: renamed from D91; moved to B.Cu
- RGB31: renamed from D92; moved to B.Cu
- RGB32: renamed from D93; moved to B.Cu
- RGB33: renamed from D94; moved to B.Cu
- RGB34: renamed from D95; moved to B.Cu
- RGB35: renamed from D96; moved to B.Cu
- RGB36: renamed from D97; moved to B.Cu
- RGB37: renamed from D98; moved to B.Cu
- RGB38: renamed from D99; moved to B.Cu
- RGB39: renamed from D100; moved to B.Cu
- RGB4: renamed from D65; moved to B.Cu
- RGB40: renamed from D101; moved to B.Cu
- RGB41: renamed from D102; moved to B.Cu
- RGB42: renamed from D103; moved to B.Cu
- RGB43: renamed from D104; moved to B.Cu
- RGB44: renamed from D105; moved to B.Cu
- RGB45: renamed from D106; moved to B.Cu
- RGB46: renamed from D107; moved to B.Cu
- RGB47: renamed from D108; moved to B.Cu
- RGB48: renamed from D109; moved to B.Cu
- RGB49: renamed from D110; moved to B.Cu
- RGB5: renamed from D66; moved to B.Cu
- RGB50: renamed from D111; moved to B.Cu
- RGB51: renamed from D112; moved to B.Cu
- RGB52: renamed from D113; moved to B.Cu
- RGB53: renamed from D114; moved to B.Cu
- RGB54: renamed from D115; moved to B.Cu
- RGB55: renamed from D116; moved to B.Cu
- RGB56: renamed from D117; moved to B.Cu
- RGB57: renamed from D118; moved to B.Cu
- RGB58: renamed from D119; moved to B.Cu
- RGB59: renamed from D120; moved to B.Cu
- RGB6: renamed from D67; moved to B.Cu
- RGB60: renamed from D121; moved to B.Cu
- RGB61: renamed from D122; moved to B.Cu
- RGB7: renamed from D68; moved to B.Cu
- RGB8: renamed from D69; moved to B.Cu
- RGB9: renamed from D70; moved to B.Cu
- moved C1 461.8 mm to (49.2, 114.1), turned to -90 degrees
- moved R1 452.9 mm to (63.2, 102.2)
- moved RGB55 441.5 mm to (51.5, 193.1), turned to 180 degrees
- moved C5 428.0 mm to (52.9, 136.4), turned to 90 degrees
- moved C2 425.5 mm to (53.1, 116.4), turned to 90 degrees
- moved RGB43 423.3 mm to (58.7, 174.3), turned to 180 degrees
- moved H4 420.3 mm to (45.9, 209.9)
- moved RGB30 415.0 mm to (58.7, 155.0), turned to 180 degrees
- moved H5 414.5 mm to (45.9, 85.7)
- moved C8 406.0 mm to (75.5, 155.0), turned to 90 degrees
- moved RGB16 405.0 mm to (61.0, 136.0), turned to 180 degrees
- moved RGB1 394.4 mm to (61.0, 116.9), turned to 180 degrees
- moved RGB44 393.8 mm to (89.6, 174.3), turned to 180 degrees
- moved RGB31 390.2 mm to (84.9, 155.0), turned to 180 degrees
- moved RGB17 383.6 mm to (84.9, 136.2), turned to 180 degrees
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Other:
- board size 341.2 x 141.6 mm -> 341.2 x 143.6 mm

Commit message: pcb done hopefully
Parts:
- added G***: LOGO, LOGO, F.Cu at (314.1, 198.0)
- added G***: LOGO, LOGO, F.Cu at (106.2, 84.3)
- R1: moved to B.Cu
- moved H3 56.8 mm to (191.6, 223.3)
- moved RGB29 0.58 mm to (346.8, 136.4), turned to 0 degrees
- moved RGB57 0.53 mm to (144.1, 203.1), turned to -12.5 degrees
- moved RGB47 0.51 mm to (148.6, 184.5), turned to -12.5 degrees
- moved RGB3 0.51 mm to (99.2, 112.7), turned to 0 degrees
- moved RGB38 0.49 mm to (254.9, 162.6), turned to 12.5 degrees
- moved RGB36 0.49 mm to (217.9, 171.0), turned to 12.5 degrees
- moved RGB37 0.49 mm to (236.4, 166.8), turned to 12.5 degrees
- moved RGB39 0.49 mm to (273.5, 158.3), turned to 12.5 degrees
- moved D57 0.48 mm to (153.9, 203.6)
- moved RGB14 0.48 mm to (327.7, 117.4), turned to 0 degrees
- moved D42 0.48 mm to (353.9, 153.6)
- moved RGB15 0.45 mm to (346.8, 117.3), turned to 0 degrees
- moved RGB2 0.45 mm to (80.1, 117.4), turned to 0 degrees
- moved RGB1 0.45 mm to (61.0, 117.4), turned to 0 degrees
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Connections:
- RGB17 pad 4: unconnected-(RGB17-DOUT-Pad4) -> Net-(RGB17-DOUT)
- RGB18 pad 2: unconnected-(RGB18-DIN-Pad2) -> Net-(RGB17-DOUT)
Routing:
- net +5V: track 0.00 -> 2469.7 mm, vias 0 -> 73
- net /ROW4: track 0.00 -> 748.9 mm, vias 0 -> 6
- net /ROW3: track 0.00 -> 721.0 mm, vias 0 -> 5
- net /ROW2: track 0.00 -> 712.7 mm, vias 0 -> 7
- net /ROW0: track 0.00 -> 703.7 mm, vias 0 -> 5
- net /ROW1: track 0.00 -> 703.6 mm, vias 0 -> 12
- net /COL0: track 0.00 -> 405.1 mm, vias 0 -> 6
- net /COL1: track 0.00 -> 361.2 mm, vias 0 -> 8
- net /COL3: track 0.00 -> 354.5 mm, vias 0 -> 10
- net Net-(RGB15-DOUT): track 0.00 -> 346.9 mm, vias 0 -> 8
- net /COL2: track 0.00 -> 346.7 mm, vias 0 -> 8
- net Net-(RGB29-DOUT): track 0.00 -> 340.8 mm, vias 0 -> 2
- net Net-(RGB42-DOUT): track 0.00 -> 338.3 mm, vias 0 -> 2
- net /COL4: track 0.00 -> 334.1 mm, vias 0 -> 8
- net Net-(RGB54-DOUT): track 0.00 -> 331.3 mm, vias 0 -> 4
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- added copper zone on B.Cu, net GND
- added copper zone on F.Cu, net GND
Other:
- board size 341.2 x 143.6 mm -> 345.9 x 162.6 mm
