File: kicad/kicad.kicad_pcb (KiCad board)
At the start: 2 copper layers, 345.9 x 162.6 mm, 211 parts, among them SW1 SW_Push, SW10 SW_Push, SW11 SW_Push, SW12 SW_Push, SW13 SW_Push, SW14 SW_Push, SW15 SW_Push, SW16 SW_Push, SW17 SW_Push, SW18 SW_Push, SW19 SW_Push, SW2 SW_Push, SW20 SW_Push, SW21 SW_Push, SW22 SW_Push, SW23 SW_Push, SW24 SW_Push, SW25 SW_Push, SW26 SW_Push, SW27 SW_Push, SW28 SW_Push, SW29 SW_Push, SW3 SW_Push, SW30 SW_Push, SW31 SW_Push, SW32 SW_Push, SW33 SW_Push, SW34 SW_Push, SW35 SW_Push, SW36 SW_Push, SW37 SW_Push, SW38 SW_Push, SW39 SW_Push, SW4 SW_Push, SW40 SW_Push, SW41 SW_Push, SW42 SW_Push, SW43 SW_Push, SW44 SW_Push, SW45 SW_Push, SW46 SW_Push, SW47 SW_Push, SW48 SW_Push, SW49 SW_Push, SW5 SW_Push, SW50 SW_Push, SW51 SW_Push, SW52 SW_Push, SW53 SW_Push, SW54 SW_Push, SW55 SW_Push, SW56 SW_Push, SW57 SW_Push, SW58 SW_Push, SW59 SW_Push, SW6 SW_Push, SW60 SW_Push, SW61 SW_Push, SW7 SW_Push, SW8 SW_Push, SW9 SW_Push

Commit message: lil changes like update footprint model and pcb changes
Parts:
- moved H6 71.2 mm to (366.0, 107.7)
- moved H3 18.8 mm to (196.3, 205.2)
- moved H4 7.95 mm to (39.7, 204.9)
- moved H5 6.25 mm to (39.9, 83.7)
- moved H1 5.36 mm to (362.2, 204.6)
- moved H2 2.38 mm to (191.6, 88.0)
- moved G*** 2.33 mm to (314.4, 195.7)
Routing:
- net +5V: track 2469.7 -> 2380.1 mm
- net GND: track 140.7 -> 208.8 mm, vias 24 -> 41
- net /ROW0: track 703.7 -> 704.1 mm, vias 5 -> 4
- net /ROW4: track 748.9 -> 749.0 mm, vias 6 -> 10
Other:
- board size 345.9 x 162.6 mm -> 340.6 x 156.5 mm
