File: kicad/rgb_matrix.kicad_sch (KiCad schematic)
At the start: 122 parts

Commit message: schematics done
Parts:
- added C1: 470u, Capacitor_Tantalum_SMD:CP_EIA-7343-31_Kemet-D_HandSolder, symbol Device:C
- added R1: 330, Resistor_SMD:R_0603_1608Metric_Pad0.98x0.95mm_HandSolder, symbol Device:R
- C10: renamed from C9; footprint (none) -> Capacitor_SMD:C_0603_1608Metric_Pad1.08x0.95mm_HandSolder
- C11: renamed from C10; footprint (none) -> Capacitor_SMD:C_0603_1608Metric_Pad1.08x0.95mm_HandSolder
- C12: renamed from C11; footprint (none) -> Capacitor_SMD:C_0603_1608Metric_Pad1.08x0.95mm_HandSolder
- C13: renamed from C12; footprint (none) -> Capacitor_SMD:C_0603_1608Metric_Pad1.08x0.95mm_HandSolder
- C14: renamed from C13; footprint (none) -> Capacitor_SMD:C_0603_1608Metric_Pad1.08x0.95mm_HandSolder
- C15: renamed from C14; footprint (none) -> Capacitor_SMD:C_0603_1608Metric_Pad1.08x0.95mm_HandSolder
- C16: renamed from C15; footprint (none) -> Capacitor_SMD:C_0603_1608Metric_Pad1.08x0.95mm_HandSolder
- C17: renamed from C16; footprint (none) -> Capacitor_SMD:C_0603_1608Metric_Pad1.08x0.95mm_HandSolder
- C18: renamed from C17; footprint (none) -> Capacitor_SMD:C_0603_1608Metric_Pad1.08x0.95mm_HandSolder
- C19: renamed from C18; footprint (none) -> Capacitor_SMD:C_0603_1608Metric_Pad1.08x0.95mm_HandSolder
- C2: renamed from C1; footprint (none) -> Capacitor_SMD:C_0603_1608Metric_Pad1.08x0.95mm_HandSolder
- C20: renamed from C19; footprint (none) -> Capacitor_SMD:C_0603_1608Metric_Pad1.08x0.95mm_HandSolder
- C21: renamed from C20; footprint (none) -> Capacitor_SMD:C_0603_1608Metric_Pad1.08x0.95mm_HandSolder
- C22: renamed from C21; footprint (none) -> Capacitor_SMD:C_0603_1608Metric_Pad1.08x0.95mm_HandSolder
- C23: renamed from C22; footprint (none) -> Capacitor_SMD:C_0603_1608Metric_Pad1.08x0.95mm_HandSolder
- C24: renamed from C23; footprint (none) -> Capacitor_SMD:C_0603_1608Metric_Pad1.08x0.95mm_HandSolder
- C25: renamed from C24; footprint (none) -> Capacitor_SMD:C_0603_1608Metric_Pad1.08x0.95mm_HandSolder
- C26: renamed from C25; footprint (none) -> Capacitor_SMD:C_0603_1608Metric_Pad1.08x0.95mm_HandSolder
- C27: renamed from C26; footprint (none) -> Capacitor_SMD:C_0603_1608Metric_Pad1.08x0.95mm_HandSolder
- C28: renamed from C27; footprint (none) -> Capacitor_SMD:C_0603_1608Metric_Pad1.08x0.95mm_HandSolder
- C29: renamed from C28; footprint (none) -> Capacitor_SMD:C_0603_1608Metric_Pad1.08x0.95mm_HandSolder
- C3: renamed from C2; footprint (none) -> Capacitor_SMD:C_0603_1608Metric_Pad1.08x0.95mm_HandSolder
- C30: renamed from C29; footprint (none) -> Capacitor_SMD:C_0603_1608Metric_Pad1.08x0.95mm_HandSolder
- C31: renamed from C30; footprint (none) -> Capacitor_SMD:C_0603_1608Metric_Pad1.08x0.95mm_HandSolder
- C32: renamed from C31; footprint (none) -> Capacitor_SMD:C_0603_1608Metric_Pad1.08x0.95mm_HandSolder
- C33: renamed from C32; footprint (none) -> Capacitor_SMD:C_0603_1608Metric_Pad1.08x0.95mm_HandSolder
- C34: renamed from C33; footprint (none) -> Capacitor_SMD:C_0603_1608Metric_Pad1.08x0.95mm_HandSolder
- C35: renamed from C34; footprint (none) -> Capacitor_SMD:C_0603_1608Metric_Pad1.08x0.95mm_HandSolder
- C36: renamed from C35; footprint (none) -> Capacitor_SMD:C_0603_1608Metric_Pad1.08x0.95mm_HandSolder
- C37: renamed from C36; footprint (none) -> Capacitor_SMD:C_0603_1608Metric_Pad1.08x0.95mm_HandSolder
- C38: renamed from C37; footprint (none) -> Capacitor_SMD:C_0603_1608Metric_Pad1.08x0.95mm_HandSolder
- C39: renamed from C38; footprint (none) -> Capacitor_SMD:C_0603_1608Metric_Pad1.08x0.95mm_HandSolder
- C4: renamed from C3; footprint (none) -> Capacitor_SMD:C_0603_1608Metric_Pad1.08x0.95mm_HandSolder
- C40: renamed from C39; footprint (none) -> Capacitor_SMD:C_0603_1608Metric_Pad1.08x0.95mm_HandSolder
- C41: renamed from C40; footprint (none) -> Capacitor_SMD:C_0603_1608Metric_Pad1.08x0.95mm_HandSolder
- C42: renamed from C41; footprint (none) -> Capacitor_SMD:C_0603_1608Metric_Pad1.08x0.95mm_HandSolder
- C43: renamed from C42; footprint (none) -> Capacitor_SMD:C_0603_1608Metric_Pad1.08x0.95mm_HandSolder
- C44: renamed from C43; footprint (none) -> Capacitor_SMD:C_0603_1608Metric_Pad1.08x0.95mm_HandSolder
- C45: renamed from C44; footprint (none) -> Capacitor_SMD:C_0603_1608Metric_Pad1.08x0.95mm_HandSolder
- C46: renamed from C45; footprint (none) -> Capacitor_SMD:C_0603_1608Metric_Pad1.08x0.95mm_HandSolder
- C47: renamed from C46; footprint (none) -> Capacitor_SMD:C_0603_1608Metric_Pad1.08x0.95mm_HandSolder
- C48: renamed from C47; footprint (none) -> Capacitor_SMD:C_0603_1608Metric_Pad1.08x0.95mm_HandSolder
- C49: renamed from C48; footprint (none) -> Capacitor_SMD:C_0603_1608Metric_Pad1.08x0.95mm_HandSolder
- C5: renamed from C4; footprint (none) -> Capacitor_SMD:C_0603_1608Metric_Pad1.08x0.95mm_HandSolder
- C50: renamed from C49; footprint (none) -> Capacitor_SMD:C_0603_1608Metric_Pad1.08x0.95mm_HandSolder
- C51: renamed from C50; footprint (none) -> Capacitor_SMD:C_0603_1608Metric_Pad1.08x0.95mm_HandSolder
- C52: renamed from C51; footprint (none) -> Capacitor_SMD:C_0603_1608Metric_Pad1.08x0.95mm_HandSolder
- C53: renamed from C52; footprint (none) -> Capacitor_SMD:C_0603_1608Metric_Pad1.08x0.95mm_HandSolder
- C54: renamed from C53; footprint (none) -> Capacitor_SMD:C_0603_1608Metric_Pad1.08x0.95mm_HandSolder
- C55: renamed from C54; footprint (none) -> Capacitor_SMD:C_0603_1608Metric_Pad1.08x0.95mm_HandSolder
- C56: renamed from C55; footprint (none) -> Capacitor_SMD:C_0603_1608Metric_Pad1.08x0.95mm_HandSolder
- C57: renamed from C56; footprint (none) -> Capacitor_SMD:C_0603_1608Metric_Pad1.08x0.95mm_HandSolder
- C58: renamed from C57; footprint (none) -> Capacitor_SMD:C_0603_1608Metric_Pad1.08x0.95mm_HandSolder
- C59: renamed from C58; footprint (none) -> Capacitor_SMD:C_0603_1608Metric_Pad1.08x0.95mm_HandSolder
- C6: renamed from C5; footprint (none) -> Capacitor_SMD:C_0603_1608Metric_Pad1.08x0.95mm_HandSolder
- C60: renamed from C59; footprint (none) -> Capacitor_SMD:C_0603_1608Metric_Pad1.08x0.95mm_HandSolder
- C61: renamed from C60; footprint (none) -> Capacitor_SMD:C_0603_1608Metric_Pad1.08x0.95mm_HandSolder
- C62: renamed from C61; footprint (none) -> Capacitor_SMD:C_0603_1608Metric_Pad1.08x0.95mm_HandSolder
- C7: renamed from C6; footprint (none) -> Capacitor_SMD:C_0603_1608Metric_Pad1.08x0.95mm_HandSolder
- C8: renamed from C7; footprint (none) -> Capacitor_SMD:C_0603_1608Metric_Pad1.08x0.95mm_HandSolder
- C9: renamed from C8; footprint (none) -> Capacitor_SMD:C_0603_1608Metric_Pad1.08x0.95mm_HandSolder
- renumbered D39 to D100, D40 to D101, D41 to D102, D42 to D103, D43 to D104, D44 to D105, D45 to D106, D46 to D107, D47 to D108, D48 to D109, D49 to D110, D50 to D111, D51 to D112, D52 to D113, D53 to D114, D54 to D115, D55 to D116, D56 to D117, D57 to D118, D58 to D119, D59 to D120, D60 to D121, D61 to D122, D1 to D62, D2 to D63, D3 to D64, D4 to D65, D5 to D66, D6 to D67, D7 to D68, D8 to D69, D9 to D70, D10 to D71, D11 to D72, D12 to D73, D13 to D74, D14 to D75, D15 to D76, D16 to D77, D17 to D78, D18 to D79, D19 to D80, D20 to D81, D21 to D82, D22 to D83, D23 to D84, D24 to D85, D25 to D86, D26 to D87, D27 to D88, D28 to D89, D29 to D90, D30 to D91, D31 to D92, D32 to D93, D33 to D94, D34 to D95, D35 to D96, D36 to D97, D37 to D98, D38 to D99
Connections:
- net 5V: now also C1.1
- net GND: now also C1.2
- net RGB: now also R1.1; no longer D62.2 (DIN)
- new net: D62.2 (DIN), R1.2

Commit message: pcb switch and diode placed but not rgbs
Parts:
- removed C10, C11, C13, C14, C15, C16, C18, C19, C20, C21, C23, C24, C25, C26, C28, C29, C3, C30, C31, C33, C34, C35, C36, C38, C39, C4, C40, C41, C43, C44, C45, C46, C48, C49, C5, C50, C51, C53, C54, C55, C56, C58, C59, C6, C60, C61, C62, C8, C9: 100n, Capacitor_SMD:C_0603_1608Metric_Pad1.08x0.95mm_HandSolder, symbol Device:C
- renumbered C42 to C10, C47 to C11, C52 to C12, C57 to C13, C7 to C3, C12 to C4, C17 to C5, C22 to C6, C27 to C7, C32 to C8, C37 to C9

Commit message: placed rgbs and relative comps in pcb
Parts:
- renumbered D62 to RGB1, D71 to RGB10, D72 to RGB11, D73 to RGB12, D74 to RGB13, D75 to RGB14, D76 to RGB15, D77 to RGB16, D78 to RGB17, D79 to RGB18, D80 to RGB19, D63 to RGB2, D81 to RGB20, D82 to RGB21, D83 to RGB22, D84 to RGB23, D85 to RGB24, D86 to RGB25, D87 to RGB26, D88 to RGB27, D89 to RGB28, D90 to RGB29, D64 to RGB3, D91 to RGB30, D92 to RGB31, D93 to RGB32, D94 to RGB33, D95 to RGB34, D96 to RGB35, D97 to RGB36, D98 to RGB37, D99 to RGB38, D100 to RGB39, D65 to RGB4, D101 to RGB40, D102 to RGB41, D103 to RGB42, D104 to RGB43, D105 to RGB44, D106 to RGB45, D107 to RGB46, D108 to RGB47, D109 to RGB48, D110 to RGB49, D66 to RGB5, D111 to RGB50, D112 to RGB51, D113 to RGB52, D114 to RGB53, D115 to RGB54, D116 to RGB55, D117 to RGB56, D118 to RGB57, D119 to RGB58, D120 to RGB59, D67 to RGB6, D121 to RGB60, D122 to RGB61, D68 to RGB7, D69 to RGB8, D70 to RGB9

Commit message: pcb done hopefully
Connections:
- net at RGB18.2 (DIN): now also RGB17.4 (DOUT)
